File: suites/drc/clearance-tolerance-is-500-nanometres/perturb/the-clean-pair-one-nanometre-closer/board.kicad_pcb (KiCad board)
At the start: 2 copper layers, 30 x 30 mm, 4 parts

Commit message: drc: keep the tolerance case to one behaviour -- four nets, not two
The two pairs shared Net-1 and GND across rows, so each net carried two pads
and the report gained two `unconnected_items` ratsnest lines that have
nothing to do with the 500 nm threshold the case pins. Each pad now takes a
net of its own and the golden is one `clearance` violation and nothing else.

  scripts/run.sh suites/drc/
    cases: 37 total, 37 clean, 0 with a failing check, 0 skipped
    PASS: 259, XFAIL: 1
  scripts/run.sh --verify-assertions
    [ASSERTED] the-clean-pair-one-nanometre-closer  moved: drc [semantic]

The case comment now records both noise sources and why each was removed --
the shared nets here, and the Reference fields lifted to (at 0 -2 0) in the
previous commit.

Co-Authored-By: Claude Opus 5 (1M context) <noreply@anthropic.com>
Connections:
- B1 pad 1: Net-1 -> Net-2
- B2 pad 1: GND -> Net-3
Changed lines of the file:
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@@
 			(size 1 1)
 			(layers "F.Cu" "F.Mask" "F.Paste")
-			(net "Net-1")
+			(net "Net-2")
 		)
 	)
@@
 			(size 1 1)
 			(layers "F.Cu" "F.Mask" "F.Paste")
-			(net "GND")
+			(net "Net-3")
 		)
 	)
