File: suites/drc/schematic-matrix-symbol-witness/board.kicad_sch (KiCad schematic)
At the start: 2 parts

Commit message: Expand KiCad DRC conformance coverage
Parts:
- R1: OracleMissing (none) -> present-only-on-symbol; OracleProbe (none) -> present-only-on-symbol
Changed lines of the file:
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@@
+			(effects (font (size 1.27 1.27)) hide)
+		)
+		(property "OracleProbe" "present-only-on-symbol"
+			(at 102 52 0)
+			(effects (font (size 1.27 1.27)) hide)
+		)
+		(property "OracleMissing" "present-only-on-symbol"
+			(at 102 53 0)
 			(effects (font (size 1.27 1.27)) hide)
 		)
